File: PCB Stuff/PumpTimerV2.kicad_pcb (KiCad board)
At the start: 4 copper layers, 65 x 50 mm, 33 parts, among them J1 1935161, J2 282856-2, J3 282856-2, J4 Conn_02x20_Odd_Even, J6 B4B-PH-SM4-TBT(LF)(SN), K1 ADW1205HLW, K2 ADW1205HLW, Q1 DMN67D7L, Q2 DMN67D7L, SW1 TL3305AF160QG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

Commit message: Start routing
Parts:
- removed the J6 at (99.5, 77.0)
- moved R8 102.4 mm to (112.4, 64.9)
- moved R3 66.7 mm to (91.4, 78.4), turned to 270 degrees
- moved C1 61.9 mm to (67.3, 72.7)
- moved R4 56.6 mm to (101.7, 83.6)
- moved U1 25.8 mm to (93.9, 80.8)
- moved J6 10.4 mm to (99.9, 77.1)
- moved R13 4.46 mm to (56.8, 82.5), turned to 180 degrees
- moved R14 1.80 mm to (46.0, 93.4)
Connections:
- U1 pad 6: +5VD -> +3V3
Routing:
- net +3V3: track 0.00 -> 33.5 mm, vias 0 -> 2
- net +BATT: track 0.00 -> 15.7 mm
- net +5VD: track 0.00 -> 10.0 mm
- net /GPIO3(SCL1): track 0.00 -> 9.84 mm, vias 0 -> 1
- net /GPIO2(SDA1): track 0.00 -> 5.53 mm
- net GND: vias 0 -> 2
- added copper zone on In1.Cu, net GND

Commit message: Routing and placement
Parts:
- removed R10, R11, R5, R6, R7, R8, R9: 49.9, Resistor_SMD:R_0603_1608Metric_Pad0.98x0.95mm_HandSolder
- moved D1 110.3 mm to (52.2, 84.3)
- moved R2 86.6 mm to (61.8, 79.5), turned to 180 degrees
- moved Q2 79.6 mm to (61.8, 84.9), turned to 270 degrees
- moved R1 70.1 mm to (80.2, 83.9)
- moved C2 67.9 mm to (67.3, 75.8)
- moved Q1 62.3 mm to (83.8, 84.9), turned to 270 degrees
- moved D3 61.9 mm to (93.0, 84.6), turned to 180 degrees
- moved D2 56.0 mm to (67.3, 78.3)
- moved R13 9.96 mm to (57.9, 72.6)
- moved R14 1.56 mm to (45.0, 92.2)
- moved SW1 1.34 mm to (44.7, 100.3)
- moved D4 1.34 mm to (44.8, 94.1)
Connections:
- net /GPIO25 renamed Net-(J4-Pad22)
- net /GPIO9(MISO) renamed Net-(J4-Pad21)
- J4 pad 7: /RLY_S -> Net-(J4-Pad7)
- J4 pad 8: Net-(J4-Pad8) -> /RLY_S
- R13 pad 1: +3V3 -> +5VD
- U1 pad 6: +3V3 -> +5VD
Routing:
- net /~BTN_RDY~: track 0.00 -> 63.3 mm, vias 0 -> 3
- net +5VD: track 10.0 -> 66.3 mm, vias 0 -> 2
- net /Reset: track 0.00 -> 47.7 mm, vias 0 -> 2
- net /Set: track 0.00 -> 44.8 mm
- net /RLY_R: track 0.00 -> 40.0 mm, vias 0 -> 2
- net Net-(R13-Pad2): track 0.00 -> 36.1 mm, vias 0 -> 2
- net /GPIO2(SDA1): track 5.53 -> 38.2 mm, vias 0 -> 2
- net /Neutral: track 0.00 -> 27.2 mm
- net /RLY_S: track 0.00 -> 23.1 mm, vias 0 -> 2
- net GND: track 0.00 -> 20.5 mm, vias 2 -> 11
- net /Line1_out: track 0.00 -> 18.5 mm
- net /Line2_in: track 0.00 -> 12.5 mm
- net /Line2_out: track 0.00 -> 11.0 mm
- net /Line1_in: track 0.00 -> 4.96 mm
- net Net-(D4-Pad2): track 0.00 -> 2.53 mm
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- added copper zone on F.Cu, net /Neutral
