File: PCB Stuff/PumpTimerV2.kicad_pcb (KiCad board)
At the start: 4 copper layers, 74 x 50 mm, 31 parts, among them J1 282856-2, J2 282856-2, J3 282856-2, J4 Conn_02x20_Odd_Even, J6 B4B-PH-SM4-TBT(LF)(SN), K1 ADW1205HLW, K2 ADW1205HLW, Q1 DMN67D7L, Q2 DMN67D7L, SW1 TL3305AF160QG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

Commit message: Potentially final routing & review. Might check things over one more time before submitting for fab
Parts:
- added C3: 100u, Capacitor_SMD:C_1206_3216Metric_Pad1.33x1.80mm_HandSolder, B.Cu at (67.3, 78.9)
- added D3: BAV5004WS-7, Diode_SMD:D_SOD-323, B.Cu at (97.8, 85.8)
- added R5: 2k2, Resistor_SMD:R_0603_1608Metric_Pad0.98x0.95mm_HandSolder, B.Cu at (87.8, 77.2)
- R1, R2: value 1k -> 10k
- renumbered D3 to D2
Connections:
- BT1 pad POS: +BATT -> Net-(BT1-PadPOS)
- D1 pad 1: /Set -> /Reset
- D2 pad 1: /Reset -> /Set
- J4 pad 12: /RLY_R -> /RLY_S
- J4 pad 7: Net-(J4-Pad7) -> /GPIO4
- J4 pad 8: /RLY_S -> /RLY_R
- K1 pad 1: /Set -> /Reset
- K1 pad 6: /Reset -> /Set
- K2 pad 1: /Set -> /Reset
- K2 pad 6: /Reset -> /Set
- Q1 pad 1: /RLY_S -> /RLY_R
- Q1 pad 3: /Set -> /Reset
- Q2 pad 1: /RLY_R -> /RLY_S
- Q2 pad 3: /Reset -> /Set
- R1 pad 2: /RLY_S -> /RLY_R
- R13 pad 2: Net-(R13-Pad2) -> /GPIO4
- R2 pad 2: /RLY_R -> /RLY_S
- SW1 pad 1: Net-(R13-Pad2) -> /GPIO4
Routing:
- net /GPIO4: track 0.00 -> 77.2 mm, vias 0 -> 3
- net Net-(R13-Pad2): track 36.1 -> 0.00 mm, vias 2 -> 0
- net /RLY_R: track 42.7 -> 24.9 mm
- net /RLY_S: track 26.6 -> 42.7 mm
- net +BATT: track 23.5 -> 11.0 mm
- net Net-(BT1-PadPOS): track 0.00 -> 10.5 mm
- net +3V3: track 31.0 -> 39.0 mm, vias 2 -> 4
- net /RTC_~INT~: track 24.1 -> 29.9 mm, vias 2 -> 3
- net +5VD: track 100.5 -> 103.6 mm
- net /Set: track 44.8 -> 47.7 mm, vias 0 -> 2
- net /Reset: track 47.7 -> 44.8 mm, vias 2 -> 0
- net GND: track 17.2 -> 18.7 mm, vias 35 -> 37
Other:
- rule pad_to_mask_clearance: 0.05 -> 0
